Commit message: Migrate tiago_robot from closed repo

File: tiago_description/gazebo/gazebo.urdf.xacro (robot description, xacro)
@@ -15,7 +15,4 @@
           <robotNamespace>/${nsp}</robotNamespace>
       </xacro:if>
-      <xacro:unless value="${is_multiple}">
-          <robotNamespace></robotNamespace>
-      </xacro:unless>
       <controlPeriod>0.001</controlPeriod>
     </plugin>

File: tiago_description/robots/tiago.urdf.xacro (robot description, xacro)
@@ -11,5 +11,5 @@
     <xacro:arg name="arm" default="true"/> <!-- true, false -->
     <xacro:arg name="wrist_model" default="wrist-2010"/>
-    <xacro:arg name="end_effector" default="pal-hey5"/> <!-- false, pal-gripper, pal-hey5, schunk-wsg-->
+    <xacro:arg name="end_effector" default="schunk-wsg-cupro"/> <!-- false, pal-gripper, pal-hey5, schunk-wsg-->
     <xacro:arg name="ft_sensor" default="schunk-ft"/> <!-- false, schunk-ft -->
     <xacro:arg name="laser_model" default="sick-571"/> <!-- false, hokuyo, sick-551, sick-561, sick-571-->
@@ -17,5 +17,8 @@
     <xacro:arg name="has_thermal_camera" default="false"/>
     <xacro:arg name="multiple" default="false"/>
+    <xacro:arg name="description_calibration_dir" default="$(find tiago_description_calibration)/urdf/calibration"/>
+    <xacro:arg name="extrinsic_calibration_dir" default="$(find tiago_description_calibration)/urdf/calibration"/>
     <xacro:arg name="namespace" default=""/>
+    <xacro:arg name="no_safety_eps" default="false"/>
     <xacro:property name="wrist_model" value="$(arg wrist_model)" />
     <xacro:property name="end_effector" value="$(arg end_effector)" />
@@ -25,8 +28,11 @@
     <xacro:property name="is_multiple" value="$(arg multiple)" />
     <xacro:property name="nsp" value="$(arg namespace)" />
-  <xacro:if value="${wrist_model not in ['wrist-2010', 'wrist-2017']}">
-    <xacro:wrong_wrist_model/>
+    <xacro:property name="no_safety_eps" value="$(arg no_safety_eps)" />
+  <xacro:if value="$(arg arm)">
+    <xacro:if value="${wrist_model not in ['wrist-2010', 'wrist-2017']}">
+      <xacro:wrong_wrist_model/>
+    </xacro:if>
   </xacro:if>
-  <xacro:if value="${end_effector not in ['false', False, 'pal-gripper', 'pal-hey5', 'schunk-wsg', 'schunk-wsg-cupro']}">
+  <xacro:if value="${end_effector not in ['false', False, 'pal-gripper', 'pal-hey5', 'schunk-wsg', 'custom', 'schunk-wsg-cupro', 'schunk-wsg-cupro-2', 'schunk-wsg-cupro-4']}">
     <xacro:wrong_end_effector/>
   </xacro:if>
@@ -47,11 +53,6 @@
    <xacro:property name="end_effector_link"       value="${'wrist_ft_tool_link' if has_ft_sensor else 'arm_tool_link'}"/>
    <xacro:property name="end_effector_name"       value="${'hand' if end_effector == 'pal-hey5' else 'gripper'}"/>
-   <xacro:if value="${wrist_model == 'wrist-2010'}">
-     <xacro:property name="wrist_6_range"           value="${ 81 if has_ft_sensor else 90 }"/>
-   </xacro:if>
-   <xacro:if value="${wrist_model == 'wrist-2017'}">
-     <xacro:property name="wrist_6_range"           value="81"/>
-   </xacro:if>
    <xacro:property name="head_link_name"          value="head_2_link"/>
+   <xacro:property name="description_calibration_dir"       value="${arg description_calibration_dir}"/>
   <!-- The following included files set up definitions of parts of the robot body -->
   <!-- Base -->
@@ -63,5 +64,5 @@
     <xacro:include filename="$(find tiago_description)/urdf/arm/arm.urdf.xacro" />
     <xacro:include filename="$(find tiago_description)/urdf/end_effector/end_effector.urdf.xacro" />
-    <xacro:include filename="$(find tiago_description_calibration)/urdf/calibration/calibration_constants.urdf.xacro" />
+  <xacro:include filename="$(arg description_calibration_dir)/calibration_constants.urdf.xacro" />
   </xacro:if>
   <!-- Force Torque sensor -->
@@ -78,7 +79,10 @@
   <xacro:base_sensors name="base" laser_model="$(arg laser_model)" sonars="true" microphone="true"/>
   <xacro:tiago_torso name="torso" parent="base_link"/>
-  <xacro:head name="head" parent="torso_lift_link" camera_model="$(arg camera_model)"/>
+  <xacro:head name="head" parent="torso_lift_link" camera_model="$(arg camera_model)"
+	  description_calibration_dir="$(arg description_calibration_dir)"
+	  extrinsic_calibration_dir="$(arg extrinsic_calibration_dir)"
+    no_safety_eps="${no_safety_eps}"/>
   <xacro:if value="${has_arm}">
-	  <xacro:tiago_arm name="arm" parent="torso_lift_link" wrist_6_range="${wrist_6_range}" reflect="1" tiago_dual="-1" arm_1_offset="${arm_1_joint_offset}" arm_2_offset="${arm_2_joint_offset}" arm_3_offset="${arm_3_joint_offset}" arm_4_offset="${arm_4_joint_offset}" arm_5_offset="${arm_5_joint_offset}" arm_6_offset="${arm_6_joint_offset}" arm_7_offset="${arm_7_joint_offset}">
+	  <xacro:tiago_arm name="arm" parent="torso_lift_link" wrist_model="${wrist_model}" has_ft_sensor="${has_ft_sensor}" reflect="1" tiago_dual="-1" arm_1_offset="${arm_1_joint_offset}" arm_2_offset="${arm_2_joint_offset}" arm_3_offset="${arm_3_joint_offset}" arm_4_offset="${arm_4_joint_offset}" arm_5_offset="${arm_5_joint_offset}" arm_6_offset="${arm_6_joint_offset}" arm_7_offset="${arm_7_joint_offset}" no_safety_eps="${no_safety_eps}">
         <origin xyz="0.15505 0.014 -0.151" rpy="0 0 ${-90 * deg_to_rad}" />
       </xacro:tiago_arm>
@@ -117,3 +121,27 @@
       </inertial>
   </link>
+  <joint name="realsense_joint" type="fixed">
+      <parent link="head_2_link"/>
+      <child link="realsense_link"/>
+      <origin xyz="0.076 0.176 0.021" rpy="-1.5707963 0.0169727 0" />
+  </joint>
+  <link name="realsense_link">
+      <inertial>
+          <origin xyz="0 0 0" rpy="0 0 0"/>
+          <mass value="0.0001" />
+          <inertia ixx="0.0001"  ixy="0"  ixz="0" iyy="0.0001" iyz="0" izz="0.0001" />
+      </inertial>
+  </link>
+  <joint name="facing_joint" type="fixed">
+      <parent link="head_2_link"/>
+      <child link="facing_link"/>
+      <origin xyz="0.0908 0.08 0" rpy="0 0 0" />
+  </joint>
+  <link name="facing_link">
+      <inertial>
+          <origin xyz="0 0 0" rpy="0 0 0"/>
+          <mass value="0.0001" />
+          <inertia ixx="0.0001"  ixy="0"  ixz="0" iyy="0.0001" iyz="0" izz="0.0001" />
+      </inertial>
+  </link>
 </robot>

File: tiago_description/urdf/arm/arm.urdf.xacro (robot description, xacro)
@@ -23,8 +23,8 @@
   <xacro:property name="arm_3_max_effort"   value="26" />
   <xacro:property name="arm_4_max_effort"   value="26" />
-  <xacro:property name="arm_eps"            value="0.07" />
   <!-- reflect: Set to 1 for a right arm, or to -1 for a left arm-->
   <!-- tiago_dual: Set to 1 for tiago dual, -1 for original tiago, changes joints 1 and 2 -->
-  <xacro:macro name="tiago_arm" params="name parent wrist_6_range reflect tiago_dual *origin arm_1_offset arm_2_offset arm_3_offset arm_4_offset arm_5_offset arm_6_offset arm_7_offset">
+  <xacro:macro name="tiago_arm" params="name parent wrist_model has_ft_sensor reflect tiago_dual *origin arm_1_offset arm_2_offset arm_3_offset arm_4_offset arm_5_offset arm_6_offset arm_7_offset no_safety_eps:=False">
+   <xacro:property name="arm_eps"       value="${0.00 if no_safety_eps else 0.07}"/>
     <!--************************-->
     <!--        SHOULDER        -->
@@ -217,5 +217,5 @@
     <!--        WRIST           -->
     <!--************************-->
-   <xacro:wrist name="${name}" parent="${name}_4_link" reflect="${reflect}" wrist_6_range="${wrist_6_range}" arm_5_offset="${arm_5_offset}" arm_6_offset="${arm_6_offset}" arm_7_offset="${arm_7_offset}"/>
+   <xacro:wrist name="${name}" parent="${name}_4_link" reflect="${reflect}" wrist_model="${wrist_model}" has_ft_sensor="${has_ft_sensor}" arm_5_offset="${arm_5_offset}" arm_6_offset="${arm_6_offset}" arm_7_offset="${arm_7_offset}"  no_safety_eps="${no_safety_eps}"/>
     <!--***********************-->
     <!--        TOOL           -->
@@ -240,8 +240,14 @@
       </collision>
     </link>
+    <xacro:if value="${wrist_model == 'wrist-2010'}">
+      <xacro:property name="tool_link_z_offset"           value="0.046"/>
+    </xacro:if>
+    <xacro:if value="${wrist_model == 'wrist-2017'}">
+     <xacro:property name="tool_link_z_offset"           value="${ 0.046 if has_ft_sensor else 0.0573 }"/>
+    </xacro:if>
     <joint name="${name}_tool_joint" type="fixed">
       <parent link="${name}_7_link" />
       <child link="${name}_tool_link" />
-      <origin xyz="0 0 ${reflect*0.046}" rpy="${90.0 * deg_to_rad} ${reflect * -90.0 * deg_to_rad} ${180 * deg_to_rad}" />
+        <origin xyz="0 0 ${reflect * tool_link_z_offset}" rpy="${90.0 * deg_to_rad} ${reflect * -90.0 * deg_to_rad} ${180 * deg_to_rad}" />
     </joint>
     <!-- extensions -->

File: tiago_description/urdf/arm/wrist.urdf.xacro (robot description, xacro)
@@ -20,6 +20,6 @@
   <xacro:property name="wrist_2_max_effort"   value="6.6" />
   <xacro:property name="wrist_3_max_effort"   value="6.6" />
-  <xacro:property name="wrist_eps"          value="0.02" />
-  <xacro:macro name="wrist" params="name parent reflect wrist_6_range arm_5_offset arm_6_offset arm_7_offset">
+  <xacro:macro name="wrist" params="name parent reflect wrist_model has_ft_sensor arm_5_offset arm_6_offset arm_7_offset no_safety_eps:=False">
+   <xacro:property name="wrist_eps"       value="${0.00 if no_safety_eps else 0.02}"/>
     <!--************************-->
     <!--        WRIST           -->
@@ -28,13 +28,21 @@
       <inertial>
         <origin xyz="0.001078 -0.000151 ${reflect * -0.077173}" rpy="0.00000 0.00000 0.00000"/>
-        <mass value="1.655819"/>
-        <inertia ixx="0.00613800000" ixy="-0.00000400000" ixz="0.00015600000"
-                 iyy="0.00564000000" iyz="0.00002200000"
-                 izz="0.00179700000"/>
+        <xacro:if value="${wrist_model == 'wrist-2010'}">
+          <mass value="1.655819"/>
+          <inertia ixx="0.00613800000" ixy="-0.00000400000" ixz="0.00015600000"
+                   iyy="0.00564000000" iyz="0.00002200000"
+                   izz="0.00179700000"/>
+        </xacro:if>
+        <xacro:if value="${wrist_model == 'wrist-2017'}">
+          <mass value="0.9359143689" />
+          <inertia ixx="0.001036187977" ixy="1.0622321E-07" ixz="1.9920336E-06"
+                   iyy="0.000794527176366096" iyz="-2.56396106998404E-07"
+                   izz="0.000439831229979178" />
+        </xacro:if>
       </inertial>
       <visual>
         <origin xyz="0 0 0" rpy="0 0 0" />
         <geometry>
-          <mesh filename="package://tiago_description/meshes/arm/arm_5.stl" scale="${reflect} ${reflect} ${reflect}"/>
+          <mesh filename="package://tiago_description/meshes/arm/arm_5-${wrist_model}.stl" scale="${reflect} ${reflect} ${reflect}"/>
         </geometry>
         <material name="LightGrey" />
@@ -43,5 +51,5 @@
         <origin xyz="0 0 0" rpy="0 0 0" />
         <geometry>
-          <mesh filename="package://tiago_description/meshes/arm/arm_5_collision.dae" scale="${reflect} ${reflect} ${reflect}"/>
+          <mesh filename="package://tiago_description/meshes/arm/arm_5_collision-${wrist_model}.dae" scale="${reflect} ${reflect} ${reflect}"/>
         </geometry>
       </collision>
@@ -62,13 +70,21 @@
       <inertial>
         <origin xyz="-0.000153 -0.003122 0.000183" rpy="0.00000 0.00000 0.00000"/>
-        <mass value="0.370063"/>
-        <inertia ixx="0.00021500000" ixy="0.00000000000" ixz="0.00000000000"
-                 iyy="0.00017000000" iyz="0.00000200000"
-                 izz="0.00017400000"/>
+        <xacro:if value="${wrist_model == 'wrist-2010'}">
+          <mass value="0.370063"/>
+          <inertia ixx="0.00021500000" ixy="0.00000000000" ixz="0.00000000000"
+                   iyy="0.00017000000" iyz="0.00000200000"
+                   izz="0.00017400000"/>
+        </xacro:if>
+        <xacro:if value="${wrist_model == 'wrist-2017'}">
+          <mass value="0.30275767222" />
+          <inertia ixx="3.29233557E-05" ixy="6.31537395E-08" ixz="-4.567124912E-11"
+                   iyy="3.85334410118923E-05" iyz="-2.01613082836742E-07"
+                   izz="3.33282849168039E-05" />
+        </xacro:if>
       </inertial>
       <visual>
         <origin xyz="0 0 0" rpy="0 0 0" />
         <geometry>
-          <mesh filename="package://tiago_description/meshes/arm/arm_6.stl" scale="${reflect} 1 1"/>
+          <mesh filename="package://tiago_description/meshes/arm/arm_6-${wrist_model}.stl" scale="${reflect} 1 1"/>
         </geometry>
         <material name="LightGrey" />
@@ -77,8 +93,14 @@
         <origin xyz="0 0 0" rpy="0 0 0" />
         <geometry>
-          <mesh filename="package://tiago_description/meshes/arm/arm_6_collision.dae" scale="${reflect} 1 1"/>
+          <mesh filename="package://tiago_description/meshes/arm/arm_6_collision-${wrist_model}.dae" scale="${reflect} 1 1"/>
         </geometry>
       </collision>
     </link>
+    <xacro:if value="${wrist_model == 'wrist-2010'}">
+      <xacro:property name="wrist_6_range"           value="${ 81 if has_ft_sensor else 90 }"/>
+    </xacro:if>
+    <xacro:if value="${wrist_model == 'wrist-2017'}">
+      <xacro:property name="wrist_6_range"           value="81"/>
+    </xacro:if>
     <joint name="${name}_6_joint" type="revolute">
       <parent link="${name}_5_link" />
@@ -96,8 +118,16 @@
       <inertial>
         <origin xyz="0.000010 -0.000003 -0.007774" rpy="0.00000 0.00000 0.00000"/>
-        <mass value="0.234252"/>
-        <inertia ixx="0.00014200000" ixy="0.00000000000" ixz="0.00000000000"
-                 iyy="0.00011300000" iyz="0.00000000000"
-                 izz="0.00005200000"/>
+        <xacro:if value="${wrist_model == 'wrist-2010'}">
+          <mass value="0.234252"/>
+          <inertia ixx="0.00014200000" ixy="0.00000000000" ixz="0.00000000000"
+                   iyy="0.00011300000" iyz="0.00000000000"
+                   izz="0.00005200000"/>
+        </xacro:if>
+        <xacro:if value="${wrist_model == 'wrist-2017'}">
+          <mass value="0.100" />
+          <inertia ixx="1.14959795E-05" ixy="-1.390727219E-07" ixz="5.930207406E-09"
+                   iyy="1.13594084240734E-05" iyz="-1.78396260812528E-08"
+                   izz="2.01898984804048E-05" />
+        </xacro:if>
       </inertial>
     </link>

File: tiago_description/urdf/end_effector/end_effector.urdf.xacro (robot description, xacro)
@@ -18,4 +18,5 @@
   -->
   <xacro:macro name="tiago_end_effector" params="name parent type reflect">
+  <!-- PAL Gripper -->
   <xacro:if value="${type == 'pal-gripper'}">
     <xacro:include filename="$(find pal_gripper_description)/urdf/gripper.urdf.xacro" />
@@ -28,5 +29,5 @@
     <xacro:include filename="$(find pal_wsg_gripper_description)/urdf/gripper.urdf.xacro" />
     <xacro:include filename="$(find pal_wsg_gripper_description)/urdf/fingertip_sensor.urdf.xacro" />
-    <xacro:pal_wsg_gripper parent="${parent}" name="${name}">
+    <xacro:pal_wsg_gripper parent="${parent}" name="${name}" lower="0.002" upper="0.034">
       <origin xyz="0.01 0 0" rpy="${90*deg_to_rad} ${90*deg_to_rad} ${-90*deg_to_rad}"/>
     </xacro:pal_wsg_gripper>
@@ -39,7 +40,64 @@
     </xacro:fingertip_sensor>
   </xacro:if>
+   <!-- Schunk + Cupro -->
+  <xacro:if value="${type == 'schunk-wsg-cupro'}">
+      <xacro:include filename="$(find pal_wsg_gripper_description)/urdf/gripper.urdf.xacro" />
+      <xacro:include filename="$(find pal_wsg_gripper_description)/urdf/fingertip_sensor.urdf.xacro" />
+      <xacro:include filename="$(find cupro_gripper_description)/urdf/gripper.urdf.xacro" />
+      <xacro:pal_wsg_gripper parent="${parent}" name="gripper" lower="0.001" upper="0.0255">
+        <origin xyz="0.01 0 0" rpy="${90*deg_to_rad} ${90*deg_to_rad} ${-90*deg_to_rad}"/>
+      </xacro:pal_wsg_gripper>
+      <xacro:cupro_gripper parent_grasp="gripper_grasping_frame" parent_l="gripper_left_finger_link" parent_r="gripper_right_finger_link" num_finger_l="1" num_finger_r="2" name="cupro">
+        <origin xyz="0 0 0" rpy="0 0 0" />
+      </xacro:cupro_gripper>
+      <!-- Fingertip sensors -->
+    <xacro:fingertip_sensor name="${name}_left" parent="${name}_left_finger">
+      <origin xyz="0.035 0 -0.1465" rpy="0 ${-90*deg_to_rad} 0"/>
+    </xacro:fingertip_sensor>
+    <xacro:fingertip_sensor name="${name}_right" parent="${name}_right_finger">
+      <origin xyz="-0.035 0 -0.1465" rpy="0 ${90*deg_to_rad} 0"/>
+    </xacro:fingertip_sensor>
+  </xacro:if>
+  <!-- Schunk + Cupro-2 -->
+  <xacro:if value="${type == 'schunk-wsg-cupro-2'}">
+      <xacro:include filename="$(find pal_wsg_gripper_description)/urdf/gripper.urdf.xacro" />
+      <xacro:include filename="$(find pal_wsg_gripper_description)/urdf/fingertip_sensor.urdf.xacro" />
+      <xacro:include filename="$(find cupro_gripper_description)/urdf/gripper.urdf.xacro" />
+      <xacro:pal_wsg_gripper parent="${parent}" name="gripper" lower="0.001" upper="0.0255">
+        <origin xyz="0.01 0 0" rpy="${90*deg_to_rad} ${90*deg_to_rad} ${-90*deg_to_rad}"/>
+      </xacro:pal_wsg_gripper>
+      <xacro:cupro_gripper parent_grasp="gripper_grasping_frame" parent_l="gripper_left_finger_link" parent_r="gripper_right_finger_link" num_finger_l="1" num_finger_r="1" name="cupro">
+        <origin xyz="0 0 0" rpy="0 0 0" />
+      </xacro:cupro_gripper>
+      <!-- Fingertip sensors -->
+    <xacro:fingertip_sensor name="${name}_left" parent="${name}_left_finger">
+      <origin xyz="0.035 0 -0.1465" rpy="0 ${-90*deg_to_rad} 0"/>
+    </xacro:fingertip_sensor>
+    <xacro:fingertip_sensor name="${name}_right" parent="${name}_right_finger">
+      <origin xyz="-0.035 0 -0.1465" rpy="0 ${90*deg_to_rad} 0"/>
+    </xacro:fingertip_sensor>
+  </xacro:if>
+  <!-- Schunk + Cupro-4 -->
+  <xacro:if value="${type == 'schunk-wsg-cupro-4'}">
+      <xacro:include filename="$(find pal_wsg_gripper_description)/urdf/gripper.urdf.xacro" />
+      <xacro:include filename="$(find pal_wsg_gripper_description)/urdf/fingertip_sensor.urdf.xacro" />
+      <xacro:include filename="$(find cupro_gripper_description)/urdf/gripper.urdf.xacro" />
+      <xacro:pal_wsg_gripper parent="${parent}" name="gripper" lower="0.001" upper="0.0255">
+        <origin xyz="0.01 0 0" rpy="${90*deg_to_rad} ${90*deg_to_rad} ${-90*deg_to_rad}"/>
+      </xacro:pal_wsg_gripper>
+      <xacro:cupro_gripper parent_grasp="gripper_grasping_frame" parent_l="gripper_left_finger_link" parent_r="gripper_right_finger_link" num_finger_l="2" num_finger_r="2" name="cupro">
+        <origin xyz="0 0 0" rpy="0 0 0" />
+      </xacro:cupro_gripper>
+      <!-- Fingertip sensors -->
+    <xacro:fingertip_sensor name="${name}_left" parent="${name}_left_finger">
+      <origin xyz="0.035 0 -0.1465" rpy="0 ${-90*deg_to_rad} 0"/>
+    </xacro:fingertip_sensor>
+    <xacro:fingertip_sensor name="${name}_right" parent="${name}_right_finger">
+      <origin xyz="-0.035 0 -0.1465" rpy="0 ${90*deg_to_rad} 0"/>
+    </xacro:fingertip_sensor>
+  </xacro:if>
   <!-- Hand -->
   <xacro:if value="${type == 'pal-hey5'}">
-    <xacro:include filename="$(find hey5_description)/urdf/hey5_hand.urdf.xacro" />
+  <xacro:include filename="$(find hey5_description)/urdf/hey5_hand.urdf.xacro" />
     <xacro:hey5_hand parent="${parent}" name="${name}" reflect="${reflect}">
       <origin xyz="0 0 0" rpy="0 0 0"/>
@@ -72,4 +130,11 @@
     </link>
   </xacro:if>
+  <!-- Custom -->
+  <xacro:if value="${type == 'custom'}">
+    <xacro:include filename="$(find custom_ee_description)/urdf/end-effector.urdf.xacro" />
+    <xacro:end_effector parent="${parent}">
+      <origin xyz="0.01 0 0" rpy="${90*deg_to_rad} ${90*deg_to_rad} ${-90*deg_to_rad}"/>
+    </xacro:end_effector>
+  </xacro:if>
   </xacro:macro>
 </robot>
