Commit message: Migrate tiago_robot from closed repo

File: tiago_description/urdf/head/head.urdf.xacro (robot description, xacro)
@@ -12,10 +12,9 @@
   <xacro:include filename="$(find tiago_description)/urdf/head/head.transmission.xacro" />
   <xacro:include filename="$(find tiago_description)/urdf/sensors/xtion_pro_live.urdf.xacro" />
-  <xacro:include filename="$(find tiago_description_calibration)/urdf/calibration/calibration_constants.urdf.xacro" />
+  <xacro:include filename="$(find tiago_description)/urdf/sensors/orbbec_astra.urdf.xacro" />
   <!--Constant parameters-->
   <xacro:property name="head_friction" value="1.0" />
   <xacro:property name="head_damping"  value="0.5" />
   <xacro:property name="head_max_vel"  value="3.0" />
-  <xacro:property name="head_eps"      value="0.07" />
   <xacro:property name="head_1_lower_limit" value="-75"/>
   <xacro:property name="head_1_upper_limit" value="75"/>
@@ -107,16 +106,47 @@
                          k_velocity="20"
                          soft_lower_limit="${head_2_lower_limit * deg_to_rad + head_eps}"
-                         soft_upper_limit="${head_2_upper_limit * deg_to_rad}" />
+                         soft_upper_limit="${head_2_upper_limit * deg_to_rad - head_eps}" />
     </joint>
     <xacro:head_transmission name="${name}" reduction="1" offset_value="${head_2_joint_offset}"/>
   </xacro:macro>
-  <xacro:macro name="head" params="name parent camera_model">
+   <!--******************************************************-->
+  <!--      Microphone + Extra Depth Cam Collision Box     -->
+  <!--*******************************************************-->
+  <xacro:macro name="head_3" params="name parent">
+    <link name="${name}_link">
+      <collision>
+        <origin xyz="0 0 0" rpy="0 0 0" />
+        <geometry>
+          <box size="0.14 0.07 0.13"/>
+        </geometry>
+      </collision>
+    </link>
+    <joint name="${name}_joint" type="fixed">
+      <parent link="${parent}"/>
+      <child link="${name}_link"/>
+      <origin xyz="0.05 0.16 0.0"  rpy="0 0 0" />
+    </joint>
+  </xacro:macro>
+  <xacro:macro name="head" params="name parent camera_model description_calibration_dir extrinsic_calibration_dir no_safety_eps:=False">
+    <xacro:property name="head_eps"      value="${0.00 if no_safety_eps else 0.07}" />
+    <!-- includes -->
+    <xacro:include filename="$(arg description_calibration_dir)/calibration_constants.urdf.xacro" />
     <xacro:head_1 name="${name}_1" parent="${parent}" />
     <xacro:head_2 name="${name}_2" parent="${name}_1_link"/>
-    <xacro:xtion_pro_live name="xtion" parent="${name}_2" camera_model="${camera_model}">
-      <origin xyz="${camera_position_x} ${camera_position_y} ${camera_position_z}" rpy="${camera_orientation_r} ${camera_orientation_p} ${camera_orientation_y}" />
-      <!-- optical origin -->
-      <origin xyz="0 0 0" rpy="${-90 * deg_to_rad} ${0 * deg_to_rad} ${-90 * deg_to_rad}" />
-    </xacro:xtion_pro_live>
+    <xacro:head_3 name="${name}_3" parent="${name}_2_link"/>
+    <xacro:if value="${camera_model == 'asus-xtion'}">
+      <xacro:xtion_pro_live name="xtion" parent="${name}_2" camera_model="${camera_model}" extrinsic_calibration_dir="${extrinsic_calibration_dir}">
+        <origin xyz="${camera_position_x} ${camera_position_y} ${camera_position_z}" rpy="${camera_orientation_r} ${camera_orientation_p} ${camera_orientation_y}" />
+        <!-- optical origin -->
+        <origin xyz="0 0 0" rpy="${-90 * deg_to_rad} ${0 * deg_to_rad} ${-90 * deg_to_rad}" />
+      </xacro:xtion_pro_live>
+    </xacro:if>
+    <xacro:if value="${camera_model in ['orbbec-astra', 'orbbec-astra-pro']}">
+      <xacro:orbbec_astra name="xtion" parent="${name}_2" camera_model="${camera_model}" extrinsic_calibration_dir="${extrinsic_calibration_dir}">
+        <origin xyz="${camera_position_x} ${camera_position_y} ${camera_position_z}" rpy="${camera_orientation_r} ${camera_orientation_p} ${camera_orientation_y}" />
+        <!-- optical origin -->
+        <origin xyz="0 0 0" rpy="${-90 * deg_to_rad} ${0 * deg_to_rad} ${-90 * deg_to_rad}" />
+      </xacro:orbbec_astra>
+    </xacro:if>
   </xacro:macro>
 </robot>

File: tiago_description/urdf/sensors/xtion_pro_live.urdf.xacro (robot description, xacro)
@@ -19,7 +19,8 @@
 <robot xmlns:xacro="http://ros.org/wiki/xacro">
   <xacro:include filename="$(find tiago_description)/urdf/sensors/openni.gazebo.xacro" />
-  <xacro:include filename="$(find tiago_description_calibration)/urdf/calibration/extrinsic_camera_calibration_constants.urdf.xacro" />
   <!-- Macro -->
-  <xacro:macro name="xtion_pro_live" params="name parent camera_model *origin *optical_origin">
+  <xacro:macro name="xtion_pro_live" params="name parent camera_model *origin *optical_origin extrinsic_calibration_dir">
+    <!-- includes -->
+    <xacro:include filename="${extrinsic_calibration_dir}/extrinsic_camera_calibration_constants.urdf.xacro" />
     <!-- frames in the center of the camera -->
     <joint name="${name}_joint" type="fixed">
